Commit message: added phantom moving link

File: serpens/src/single_joint/urdf/snake_joint.xacro (robot description, xacro)
@@ -106,4 +106,52 @@
         </inertial>
     </link>
+    <!--add a phantom of the moving link to display the desired position-->
+    <link name="pivot_phantom">
+        <visual>
+            <origin xyz="0 0 0" rpy="0 0 0" />
+            <geometry>
+                <cylinder radius="${RADIUS_5}" length="${LENGTH_5}" />
+            </geometry>
+        </visual>
+        <collision>
+            <origin xyz="0 0 0" rpy="0 0 0" />
+            <geometry>
+                <cylinder radius="${RADIUS_5}" length="${LENGTH_5}" />
+            </geometry>
+        </collision>
+        <inertial>
+            <origin xyz="0 0 0" rpy="0 0 0" />
+            <mass value="${MASS_3}"/>
+            <inertia ixx="${((MASS_3 * (LENGTH_5 * LENGTH_5)) / 12) + (MASS_3 * (RADIUS_5 * RADIUS_5)) / 4}" ixy="0.0" ixz="0.0"
+                     iyy="${((MASS_3 * (LENGTH_5 * LENGTH_5)) / 12) + (MASS_3 * (RADIUS_5 * RADIUS_5)) / 4}" iyz="0.0"
+                     izz="${(MASS_3 * (RADIUS_5 * RADIUS_5)) / 2}"/>
+        </inertial>
+    </link>
+    <link name="moving_link_phantom">
+        <inertial>
+            <origin xyz="${(LENGTH_4 / 2) + (RADIUS_5 / 2)} 0 0" rpy="0 ${M_PI / 2} 0" />
+            <mass value= "1.0"/>
+            <inertia ixx="0.0" ixy="0.0" ixz="0.0"
+                     iyy="0.0" iyz="0.0"
+                     izz="0.0"/>
+        </inertial>
+        <visual>
+            <origin xyz="${(LENGTH_4 / 2) + (RADIUS_5 / 2)} 0 0" rpy="0 ${M_PI / 2} 0" />
+            <geometry>
+                <cylinder radius="${RADIUS_4}" length="${LENGTH_4}" />
+            </geometry>
+            <material name="MyGreen">
+                <ambient>0 1 0 1</ambient>
+                <diffuse>0 1 0 1</diffuse>
+                <color rgba="0 1.0 0.5 1.0"/>
+            </material>
+        </visual>
+        <collision>
+            <origin xyz="100000 0 0" rpy="0 ${M_PI / 2} 0" />
+            <geometry>
+                <cylinder radius="${RADIUS_4}" length="${LENGTH_4}" />
+            </geometry>
+        </collision>
+    </link>
     <joint name="world_to_base" type="fixed">
         <parent link="world"/>
@@ -129,4 +177,20 @@
         <limit effort="10" lower="-0.4" upper="0.4" velocity="1" />
     </joint>
+    <!--add a phantom of the moving link to display the desired position-->
+    <joint name="fixated_to_pivot_phantom" type="revolute">
+        <parent link="fixated_link" />
+        <child link="pivot_phantom" />
+        <axis xyz="0 0 1" />
+        <origin xyz="0 0 ${LENGTH_4}" rpy="0 -${M_PI / 2} 0"/>
+        <limit effort="1000.0" lower="${-M_PI / 2}" upper="${M_PI / 2}" velocity="1.0" />
+    </joint>
+    <joint name="pivot_to_moving_link_phantom" type="revolute">
+        <parent link="pivot_phantom" />
+        <child link="moving_link_phantom" />
+        <axis xyz="0 0 1" />
+        <origin xyz="0 0 0" />
+        <dynamics damping="1"/>
+        <limit effort="10" lower="-0.4" upper="0.4" velocity="1" />
+    </joint>
     <transmission name="motor_tran">
         <type>transmission_interface/SimpleTransmission</type>
@@ -149,3 +213,24 @@
         </actuator>
     </transmission>
+<!--Added for phantom-->
+    <transmission name="motor_tran_phantom">
+        <type>transmission_interface/SimpleTransmission</type>
+        <joint name="fixated_to_pivot_phantom">
+            <hardwareInterface>hardware_interface/EffortJointInterface</hardwareInterface>
+        </joint>
+        <actuator name="motor_phantom">
+            <hardwareInterface>hardware_interface/EffortJointInterface</hardwareInterface>
+            <mechanicalReduction>1</mechanicalReduction>
+        </actuator>
+    </transmission>
+    <transmission name="spring_tran_phantom">
+        <type>transmission_interface/SimpleTransmission</type>
+        <joint name="pivot_to_moving_link_phantom">
+            <hardwareInterface>hardware_interface/EffortJointInterface</hardwareInterface>
+        </joint>
+        <actuator name="spring_phantom">
+            <hardwareInterface>hardware_interface/EffortJointInterface</hardwareInterface>
+            <mechanicalReduction>1</mechanicalReduction>
+        </actuator>
+    </transmission>
 </robot>

Commit message: with correct spring

File: serpens/src/single_joint/urdf/snake_joint.xacro (robot description, xacro)
@@ -107,4 +107,5 @@
     </link>
     <!--add a phantom of the moving link to display the desired position-->
+    <!--
     <link name="pivot_phantom">
         <visual>
@@ -154,4 +155,5 @@
         </collision>
     </link>
+-->
     <joint name="world_to_base" type="fixed">
         <parent link="world"/>
@@ -167,15 +169,18 @@
         <axis xyz="0 0 1" />
         <origin xyz="0 0 ${LENGTH_4}" rpy="0 -${M_PI / 2} 0"/>
+        <dynamics damping="1"/>
         <limit effort="1000.0" lower="${-M_PI / 2}" upper="${M_PI / 2}" velocity="1.0" />
     </joint>
-    <joint name="pivot_to_moving_link" type="revolute">
+    <joint name="pivot_to_moving_link" type="fixed">
         <parent link="pivot" />
         <child link="moving_link" />
+        <!--
         <axis xyz="0 0 1" />
         <origin xyz="0 0 0" />
         <dynamics damping="1"/>
         <limit effort="10" lower="-0.4" upper="0.4" velocity="1" />
-    </joint>
-    <!--add a phantom of the moving link to display the desired position-->
+        -->
+    </joint>
+    <!--add a phantom of the moving link to display the desired position
     <joint name="fixated_to_pivot_phantom" type="revolute">
         <parent link="fixated_link" />
@@ -190,7 +195,8 @@
         <axis xyz="0 0 1" />
         <origin xyz="0 0 0" />
-        <dynamics damping="1"/>
+        <dynamics damping="100"/>
         <limit effort="10" lower="-0.4" upper="0.4" velocity="1" />
     </joint>
+    -->
     <transmission name="motor_tran">
         <type>transmission_interface/SimpleTransmission</type>
@@ -203,4 +209,5 @@
         </actuator>
     </transmission>
+    <!--
     <transmission name="spring_tran">
         <type>transmission_interface/SimpleTransmission</type>
@@ -213,5 +220,7 @@
         </actuator>
     </transmission>
+-->
 <!--Added for phantom-->
+<!--
     <transmission name="motor_tran_phantom">
         <type>transmission_interface/SimpleTransmission</type>
@@ -234,3 +243,4 @@
         </actuator>
     </transmission>
+-->
 </robot>

Commit message: Green joint is back

File: serpens/src/single_joint/urdf/snake_joint.xacro (robot description, xacro)
@@ -107,5 +107,4 @@
     </link>
     <!--add a phantom of the moving link to display the desired position-->
-    <!--
     <link name="pivot_phantom">
         <visual>
@@ -155,5 +154,4 @@
         </collision>
     </link>
--->
     <joint name="world_to_base" type="fixed">
         <parent link="world"/>
@@ -182,5 +180,5 @@
         -->
     </joint>
-    <!--add a phantom of the moving link to display the desired position
+    <!--add a phantom of the moving link to display the desired position-->
     <joint name="fixated_to_pivot_phantom" type="revolute">
         <parent link="fixated_link" />
@@ -190,11 +188,7 @@
         <limit effort="1000.0" lower="${-M_PI / 2}" upper="${M_PI / 2}" velocity="1.0" />
     </joint>
-    <joint name="pivot_to_moving_link_phantom" type="revolute">
+    <joint name="pivot_to_moving_link_phantom" type="fixed">
         <parent link="pivot_phantom" />
         <child link="moving_link_phantom" />
-        <axis xyz="0 0 1" />
-        <origin xyz="0 0 0" />
-        <dynamics damping="100"/>
-        <limit effort="10" lower="-0.4" upper="0.4" velocity="1" />
     </joint>
     -->
@@ -222,15 +216,15 @@
 -->
 <!--Added for phantom-->
+    <transmission name="motor_tran_phantom">
+        <type>transmission_interface/SimpleTransmission</type>
+        <joint name="fixated_to_pivot_phantom">
+            <hardwareInterface>hardware_interface/EffortJointInterface</hardwareInterface>
+        </joint>
+        <actuator name="motor_phantom">
+            <hardwareInterface>hardware_interface/EffortJointInterface</hardwareInterface>
+            <mechanicalReduction>1</mechanicalReduction>
+        </actuator>
+    </transmission>
 <!--
-    <transmission name="motor_tran_phantom">
-        <type>transmission_interface/SimpleTransmission</type>
-        <joint name="fixated_to_pivot_phantom">
-            <hardwareInterface>hardware_interface/EffortJointInterface</hardwareInterface>
-        </joint>
-        <actuator name="motor_phantom">
-            <hardwareInterface>hardware_interface/EffortJointInterface</hardwareInterface>
-            <mechanicalReduction>1</mechanicalReduction>
-        </actuator>
-    </transmission>
     <transmission name="spring_tran_phantom">
         <type>transmission_interface/SimpleTransmission</type>
